File: schema/led-dimmer.kicad_pcb (KiCad board)
At the start: 2 copper layers, 70 x 50 mm, 20 parts, among them IC1 ATTINY85-P, K1 CONN_3, P1 CONN_2, P2 CONN_3, Q1 BS107, Q2 IRF9530, U1 LM7805

Commit message: New PCB which allows to connect bypassing LC filter
Parts:
- moved Q1 1.30 mm to (34.8, 50.5)
Routing:
- net Net-(Q1-PadG): track 6.35 -> 13.1 mm
- net Net-(Q1-PadD): track 14.3 -> 11.3 mm
Changed lines of the file:
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@@
   (general
     (links 29)
-    (no_connects 1)
+    (no_connects 0)
     (area 15.174999 12.33705 85.325001 67.83605)
     (thickness 1.6)
     (drawings 7)
-    (tracks 55)
+    (tracks 57)
     (zones 0)
     (modules 20)
@@
   )
   (module TO92DGS (layer F.Cu)
-    (at 33.46 50.62)
+    (at 34.75 50.5)
     (descr "Transistor TO92 brochage type BC237")
     (tags "TR TO92")
@@
   (segment (start 30.68 31.57) (end 32.19 31.57) (width 0.3) (layer B.Cu) (net 5))
   (segment (start 19.49 43) (end 19.49 39.19) (width 0.3) (layer B.Cu) (net 6))
-  (segment (start 36 43) (end 36 48.08) (width 0.3) (layer B.Cu) (net 10))
-  (segment (start 36 48.08) (end 34.73 49.35) (width 0.3) (layer B.Cu) (net 10))
-  (segment (start 34.73 49.35) (end 34.73 51.23) (width 0.3) (layer B.Cu) (net 10))
-  (segment (start 36.06 52.56) (end 39.75 52.56) (width 0.3) (layer B.Cu) (net 10))
-  (segment (start 34.73 51.23) (end 36.06 52.56) (width 0.3) (layer B.Cu) (net 10))
-  (segment (start 32.19 43) (end 32.19 49.35) (width 0.3) (layer B.Cu) (net 11))
+  (segment (start 36.02 43.02) (end 36 43) (width 0.3) (layer B.Cu) (net 10))
+  (segment (start 36.02 49.23) (end 36.02 43.02) (width 0.3) (layer B.Cu) (net 10))
+  (segment (start 36.42 49.23) (end 39.75 52.56) (width 0.3) (layer B.Cu) (net 10))
+  (segment (start 36.02 49.23) (end 36.42 49.23) (width 0.3) (layer B.Cu) (net 10))
+  (segment (start 32.19 47.94) (end 33.48 49.23) (width 0.3) (layer B.Cu) (net 11))
+  (segment (start 32.19 43) (end 32.19 47.94) (width 0.3) (layer B.Cu) (net 11))
+  (segment (start 29.02 53.69) (end 33.48 49.23) (width 0.3) (layer B.Cu) (net 11))
+  (segment (start 29 53.69) (end 29.02 53.69) (width 0.3) (layer B.Cu) (net 11))
   (segment (start 39.75 44.94) (end 42.19 44.94) (width 0.3) (layer B.Cu) (net 12))
   (segment (start 44.5 48.5) (end 46.71 48.5) (width 0.3) (layer B.Cu) (net 12))
